Commit message: collisions now work, contact sensor does not, added work piece to model

File: panda_table_description/urdf/panda_table.urdf.xacro (robot description, xacro)
@@ -6,6 +6,6 @@
   <xacro:include filename="$(find franka_description)/robots/hand.xacro"/>
   <!-- for simulation -->
-  <xacro:include filename="$(find franka_description)/robots/panda.gazebo.xacro"/>
   <xacro:include filename="$(find franka_description)/robots/panda.transmission.xacro"/>
+  <xacro:include filename="$(find panda_table_description)/urdf/panda_table.gazebo.xacro"/>
   <!-- end for simulation -->
   <xacro:panda_arm connected_to="mount_flange_link" xyz="0.0 0.0 0.0" rpy="0 0 ${pi}" />
@@ -14,8 +14,33 @@
   </xacro:if>
   <xacro:unless value="$(arg load_gripper)">
+   <link name="tool">
+     <inertial>
+       <mass value="0.642"/>
+       <inertia ixx="0.001" ixy="0" ixz="0" iyy="0.001" iyz="0" izz="0.001" />
+       <origin/>
+     </inertial>
+     <visual>
+       <origin xyz="0 0 -0.15" rpy="0 0 0" />
+       <geometry>
+         <cylinder radius="0.0085" length="0.3" />
+       </geometry>
+       <material name="orange"/>
+     </visual>
+     <collision name="tool_collision">
+       <origin xyz="0 0 -0.15" rpy="0 0 0" />
+       <geometry>
+         <cylinder radius="0.0085" length="0.3" />
+       </geometry>
+     </collision>
+   </link>
+     <joint name="tool_joint" type="fixed">
+       <parent link="panda_link8" />
+       <child link = "tool" />
+       <origin xyz="0.0 0.0 0.3" rpy="0.0 0.0 0.0" />
+     </joint>
   </xacro:unless>
   <!-- for simulation -->
   <xacro:arg name="robot_name" default="panda"/>
-  <xacro:panda_gazebo robot_name="$(arg robot_name)" load_gripper="$(arg load_gripper)" />
+  <xacro:panda_table_gazebo robot_name="$(arg robot_name)" load_gripper="$(arg load_gripper)" />
   <xacro:panda_transmission robot_name="$(arg robot_name)" load_gripper="$(arg load_gripper)" />
   <!-- end for simulation -->
@@ -77,4 +102,18 @@
     </collision>
    </link>
+   <link name="work_piece">
+    <visual>
+      <geometry>
+	<mesh filename="package://panda_table_description/meshes/work_piece.stl" scale="0.001 0.001 0.001"/>
+      </geometry>
+      <origin rpy="0 1.5707 0" xyz="0.0 0.0 0.0" />
+    </visual>
+    <collision>
+      <geometry>
+	<mesh filename="package://panda_table_description/meshes/work_piece.stl" scale="0.001 0.001 0.001"/>
+      </geometry>
+      <origin rpy="0 1.5707 0" xyz="0.0 0.0 0.0" />
+    </collision>
+   </link>
   <joint name="world_joint" type="fixed">
     <parent link="world" />
@@ -97,3 +136,8 @@
     <origin xyz="-0.45 -0.505 0.7" rpy="0.0 0.0 0.0" />
   </joint>
+  <joint name="table_wp" type="fixed">
+    <parent link="table" />
+    <child link = "work_piece" />
+    <origin xyz="0.45 0.105 0.72" rpy="0.0 0.0 0.0" />
+  </joint>
 </robot>

Commit message: added 'origin' values to xacro file necessary for 'kdl_parser_py' to not crash - continuation of work on resolved rate motion control

File: panda_table_description/urdf/panda_table.urdf.xacro (robot description, xacro)
@@ -18,5 +18,5 @@
        <mass value="0.642"/>
        <inertia ixx="0.001" ixy="0" ixz="0" iyy="0.001" iyz="0" izz="0.001" />
-       <origin/>
+       <origin xyz="0 0 0" rpy="0 0 0" />
      </inertial>
      <visual>
@@ -64,5 +64,5 @@
        <mass value="0.01"/>
        <inertia ixx="0.001" ixy="0" ixz="0" iyy="0.001" iyz="0" izz="0.001" />
-       <origin/>
+       <origin xyz="0 0 0" rpy="0 0 0" />
      </inertial>
      <visual>

Commit message: fixed urdf table representation and added board and camera support
Former-commit-id: da53235a04b8b65c4236c4be065126a9ae5e8ae4 [formerly af1a37a5d883ab937b80917b151e1196b6ba6ed1]
Former-commit-id: b2faaa5d4c7618a269583383f51bebe011e54c09

File: panda_table_description/urdf/panda_table.urdf.xacro (robot description, xacro)
@@ -116,5 +116,19 @@
     </collision>
    </link>
-   <link name="work_piece">
+   <link name="camera_long_support">
+    <visual>
+      <geometry>
+	<box size="1.8 0.08 0.04" />
+      </geometry>
+      <origin rpy="0 0 0" xyz="0.0 0.0 0.02" />
+    </visual>
+    <collision>
+      <geometry>
+	<box size="1.8 0.08 0.04" />
+      </geometry>
+      <origin rpy="0 0 0" xyz="0.0 0.0 0.02" />
+    </collision>
+   </link>
+   <!-- <link name="work_piece">
     <visual>
       <geometry>
@@ -129,5 +143,5 @@
       <origin rpy="0 1.5707 0" xyz="0.0 0.0 0.0" />
     </collision>
-   </link>
+   </link> -->
   <joint name="world_joint" type="fixed">
     <parent link="world" />
@@ -138,6 +152,5 @@
     <parent link="table" />
     <child link = "mount_flange_link" />
-    <origin xyz="0.0 0.425 0.7" rpy="0.0 0.0 1.5707" />
-    <!-- <origin xyz="0.0 0.414 0.7" rpy="0.0 0.0 1.5707" /> -->
+    <origin xyz="0.02 0.305 0.7" rpy="0.0 0.0 1.5707" />
   </joint>
   <joint name="table_board" type="fixed">
@@ -145,4 +158,9 @@
     <child link = "board" />
     <origin xyz="0.4 -0.230 0.715" rpy="0.0 0.0 0.0" />
+  </joint>
+  <joint name="table_camera_long_support" type="fixed">
+    <parent link="table" />
+    <child link = "camera_long_support" />
+    <origin xyz="0.4 -0.510 1.215" rpy="0.0 0.0 0.0" />
   </joint>
   <joint name="table_column1" type="fixed">
@@ -156,8 +174,8 @@
     <origin xyz="-0.45 -0.505 0.7" rpy="0.0 0.0 0.0" />
   </joint>
-  <joint name="table_wp" type="fixed">
+  <!-- <joint name="table_wp" type="fixed">
     <parent link="table" />
     <child link = "work_piece" />
     <origin xyz="0.45 0.105 0.72" rpy="0.0 0.0 0.0" />
-  </joint>
+  </joint> -->
 </robot>
