Commit message: added board to urdf model - initial work on push trajectory
Former-commit-id: fe6dbc80c4983c6ea0c6fe8cea659536c28b0917 [formerly 3e3ff4fda304843e7b00f8d4fb34632a15a2ad42]
Former-commit-id: 7bf3ccf44b2b9994a28e60952f143ded4e3fdd9e

File: panda_table_description/urdf/panda_table.gazebo.xacro (robot description, xacro)
@@ -106,4 +106,10 @@
 	    <self_collide>true</self_collide>
         </gazebo>
+ <gazebo reference="board">
+            <material>Gazebo/Grey</material>
+            <mu1>0.2</mu1>
+            <mu2>0.2</mu2>
+	    <self_collide>true</self_collide>
+        </gazebo>
  <gazebo reference="column1">
             <material>Gazebo/Grey</material>

File: panda_table_description/urdf/panda_table.urdf.xacro (robot description, xacro)
@@ -58,4 +58,18 @@
       </geometry>
       <origin rpy="0 0 0" xyz="0 0 0.35" />
+    </collision>
+   </link>
+  <link name="board">
+    <visual>
+      <geometry>
+	<box size="2.0 0.45 0.03" />
+      </geometry>
+      <origin rpy="0 0 0" xyz="0 0 0" />
+    </visual>
+    <collision>
+      <geometry>
+	<box size="2.0 0.45 0.03" />
+      </geometry>
+      <origin rpy="0 0 0" xyz="0 0 0" />
     </collision>
    </link>
@@ -125,4 +139,10 @@
     <child link = "mount_flange_link" />
     <origin xyz="0.0 0.425 0.7" rpy="0.0 0.0 1.5707" />
+    <!-- <origin xyz="0.0 0.414 0.7" rpy="0.0 0.0 1.5707" /> -->
+  </joint>
+  <joint name="table_board" type="fixed">
+    <parent link="table" />
+    <child link = "board" />
+    <origin xyz="0.4 -0.230 0.715" rpy="0.0 0.0 0.0" />
   </joint>
   <joint name="table_column1" type="fixed">

Commit message: modifications for simulation of panda to make it more stable. second feature is updates to how the task dynamics plugin makes sure that destructors are called correctly

File: panda_table_description/urdf/panda_table.gazebo.xacro (robot description, xacro)
@@ -2,4 +2,5 @@
 <robot xmlns:xacro="http://www.ros.org/wiki/xacro">
     <xacro:macro name="panda_table_gazebo" params="robot_name:='panda' load_gripper:='true'">
+	    <!-- set the model to be static, enable self collision -->
         <!-- Link0 -->
         <gazebo reference="${robot_name}_link0">
@@ -7,4 +8,5 @@
             <mu1>0.2</mu1>
             <mu2>0.2</mu2>
+	    <self_collide>true</self_collide>
         </gazebo>
         <!-- Link1 -->
@@ -13,4 +15,5 @@
             <mu1>0.2</mu1>
             <mu2>0.2</mu2>
+	    <self_collide>true</self_collide>
         </gazebo>
         <!-- Link2 -->
@@ -19,4 +22,5 @@
             <mu1>0.2</mu1>
             <mu2>0.2</mu2>
+	    <self_collide>true</self_collide>
         </gazebo>
         <!-- Link3 -->
@@ -25,4 +29,5 @@
             <mu1>0.2</mu1>
             <mu2>0.2</mu2>
+	    <self_collide>true</self_collide>
         </gazebo>
         <!-- Link4 -->
@@ -31,4 +36,5 @@
             <mu1>0.2</mu1>
             <mu2>0.2</mu2>
+	    <self_collide>true</self_collide>
         </gazebo>
         <!-- Link5 -->
@@ -37,4 +43,5 @@
             <mu1>0.2</mu1>
             <mu2>0.2</mu2>
+	    <self_collide>true</self_collide>
         </gazebo>
         <!-- Link6 -->
@@ -43,4 +50,5 @@
             <mu1>0.2</mu1>
             <mu2>0.2</mu2>
+	    <self_collide>true</self_collide>
         </gazebo>
         <!-- Link7 -->
@@ -71,4 +79,5 @@
             <mu1>0.2</mu1>
             <mu2>0.2</mu2>
+	    <self_collide>true</self_collide>
         </gazebo>
         <!-- LinkLeftFinger -->
@@ -77,4 +86,5 @@
             <mu1>0.2</mu1>
             <mu2>0.2</mu2>
+	    <self_collide>true</self_collide>
         </gazebo>
 	</xacro:if>
@@ -105,4 +115,5 @@
             <mu2>0.2</mu2>
 	    <self_collide>true</self_collide>
+	    <static>true</static>
         </gazebo>
  <gazebo reference="column1">

File: panda_table_description/urdf/panda_table.urdf.xacro (robot description, xacro)
@@ -47,4 +47,9 @@
   <link name="world" />
   <link name="table">
+     <inertial>
+       <mass value="200.0"/>
+       <inertia ixx="10.0" ixy="0" ixz="0" iyy="10.0" iyz="0" izz="10.0" />
+       <origin/>
+     </inertial>
     <visual>
       <geometry>
@@ -74,5 +79,4 @@
      </visual>
    </link>
-   <!--
     <link name="column1">
      <visual>
@@ -81,4 +85,5 @@
        </geometry>
        <origin rpy="0 0 0" xyz="0.0 0.0 0.2575" />
+       <material name="orange"/>
      </visual>
      <collision>
@@ -95,4 +100,5 @@
        </geometry>
        <origin rpy="0 0 0" xyz="0.0 0.0 0.2575" />
+       <material name="orange"/>
      </visual>
      <collision>
@@ -103,19 +109,4 @@
      </collision>
     </link>
-    <link name="work_piece">
-     <visual>
-       <geometry>
-     <mesh filename="package://panda_table_description/meshes/work_piece.stl" scale="0.001 0.001 0.001"/>
-       </geometry>
-       <origin rpy="0 1.5707 0" xyz="0.0 0.0 0.0" />
-     </visual>
-     <collision>
-       <geometry>
-     <mesh filename="package://panda_table_description/meshes/work_piece.stl" scale="0.001 0.001 0.001"/>
-       </geometry>
-       <origin rpy="0 1.5707 0" xyz="0.0 0.0 0.0" />
-     </collision>
-    </link>
-    -->
   <joint name="world_joint" type="fixed">
     <parent link="world" />
@@ -128,5 +119,4 @@
     <origin xyz="0.0 0.425 0.7" rpy="0.0 0.0 1.5707" />
   </joint>
-  <!--
   <joint name="table_column1" type="fixed">
     <parent link="table" />
@@ -139,4 +129,5 @@
     <origin xyz="-0.45 -0.505 0.7" rpy="0.0 0.0 0.0" />
   </joint>
+  <!--
   <joint name="table_wp" type="fixed">
     <parent link="table" />

Commit message: description files

File: panda_table_description/urdf/panda_table.gazebo.xacro (robot description, xacro)
@@ -7,4 +7,5 @@
             <mu1>0.2</mu1>
             <mu2>0.2</mu2>
+            <self_collide>true</self_collide>
         </gazebo>
         <!-- Link1 -->
@@ -13,4 +14,5 @@
             <mu1>0.2</mu1>
             <mu2>0.2</mu2>
+            <self_collide>true</self_collide>
         </gazebo>
         <!-- Link2 -->
@@ -19,4 +21,5 @@
             <mu1>0.2</mu1>
             <mu2>0.2</mu2>
+            <self_collide>true</self_collide>
         </gazebo>
         <!-- Link3 -->
@@ -25,4 +28,5 @@
             <mu1>0.2</mu1>
             <mu2>0.2</mu2>
+            <self_collide>true</self_collide>
         </gazebo>
         <!-- Link4 -->
@@ -31,4 +35,5 @@
             <mu1>0.2</mu1>
             <mu2>0.2</mu2>
+            <self_collide>true</self_collide>
         </gazebo>
         <!-- Link5 -->
@@ -37,4 +42,5 @@
             <mu1>0.2</mu1>
             <mu2>0.2</mu2>
+            <self_collide>true</self_collide>
         </gazebo>
         <!-- Link6 -->
@@ -43,4 +49,5 @@
             <mu1>0.2</mu1>
             <mu2>0.2</mu2>
+            <self_collide>true</self_collide>
         </gazebo>
         <!-- Link7 -->
@@ -105,5 +112,6 @@
             <mu2>0.2</mu2>
 	    <self_collide>true</self_collide>
-        </gazebo>
+        <static>true</static>
+    </gazebo>
  	<gazebo reference="column1">
             <material>Gazebo/Grey</material>

File: panda_table_description/urdf/panda_table.urdf.xacro (robot description, xacro)
@@ -7,4 +7,5 @@
   <xacro:include filename="$(find franka_description)/robots/panda.transmission.xacro"/>
   <xacro:include filename="$(find panda_table_description)/urdf/panda_table.gazebo.xacro"/>
+  <xacro:include filename="$(find panda_table_description)/urdf/table.urdf.xacro"/>
   <!-- end for simulation -->
   <xacro:panda_arm connected_to="mount_flange_link" xyz="0.0 0.0 0.0" rpy="0 0 ${pi}" />
@@ -44,19 +45,21 @@
   <xacro:panda_transmission robot_name="$(arg robot_name)" load_gripper="$(arg load_gripper)" />
   <!-- end for simulation -->
-  <link name="world" />
-  <link name="table">
-    <visual>
-      <geometry>
-	<box size="1.0 1.11 0.7" />
-      </geometry>
-      <origin rpy="0 0 0" xyz="0 0 0.35" />
-    </visual>
-    <collision>
-      <geometry>
-	<box size="1.0 1.11 0.7" />
-      </geometry>
-      <origin rpy="0 0 0" xyz="0 0 0.35" />
-    </collision>
-   </link>
+  <!--
+    <link name="world" />
+    <link name="table">
+      <visual>
+        <geometry>
+      <box size="1.0 1.11 0.7" />
+        </geometry>
+        <origin rpy="0 0 0" xyz="0 0 0.35" />
+      </visual>
+      <collision>
+        <geometry>
+      <box size="1.0 1.11 0.7" />
+        </geometry>
+        <origin rpy="0 0 0" xyz="0 0 0.35" />
+      </collision>
+     </link>
+  -->
    <link name="mount_flange_link">
      <inertial>
@@ -73,69 +76,5 @@
      </visual>
    </link>
-    <!--
-    <link name="box">
-     <visual>
-       <geometry>
-     <box size="0.04 0.04 0.04" />
-       </geometry>
-       <origin rpy="0 0 0" xyz="0.0 0.0 0.2575" />
-     </visual>
-     <collision>
-       <geometry>
-     <box size="0.1 0.1 0.1" />
-       </geometry>
-       <origin rpy="0 0 0" xyz="0.0 0.0 0.2575" />
-     </collision>
-    </link>
-    <joint name="table_box" type="fixed">
-      <parent link="table" />
-      <child link = "box" />
-      <origin xyz="-0.2 0.0 0.5325" rpy="0.0 0.0 0.0" />
-    </joint>
-    -->
-   <!--
-    <link name="column1">
-     <visual>
-       <geometry>
-     <box size="0.1 0.1 0.515" />
-       </geometry>
-       <origin rpy="0 0 0" xyz="0.0 0.0 0.2575" />
-     </visual>
-     <collision>
-       <geometry>
-     <box size="0.1 0.1 0.515" />
-       </geometry>
-       <origin rpy="0 0 0" xyz="0.0 0.0 0.2575" />
-     </collision>
-    </link>
-    <link name="column2">
-     <visual>
-       <geometry>
-     <box size="0.1 0.1 0.515" />
-       </geometry>
-       <origin rpy="0 0 0" xyz="0.0 0.0 0.2575" />
-     </visual>
-     <collision>
-       <geometry>
-     <box size="0.1 0.1 0.515" />
-       </geometry>
-       <origin rpy="0 0 0" xyz="0.0 0.0 0.2575" />
-     </collision>
-    </link>
-    <link name="work_piece">
-     <visual>
-       <geometry>
-     <mesh filename="package://panda_table_description/meshes/work_piece.stl" scale="0.001 0.001 0.001"/>
-       </geometry>
-       <origin rpy="0 1.5707 0" xyz="0.0 0.0 0.0" />
-     </visual>
-     <collision>
-       <geometry>
-     <mesh filename="package://panda_table_description/meshes/work_piece.stl" scale="0.001 0.001 0.001"/>
-       </geometry>
-       <origin rpy="0 1.5707 0" xyz="0.0 0.0 0.0" />
-     </collision>
-    </link>
-    -->
+<!--
   <joint name="world_joint" type="fixed">
     <parent link="world" />
@@ -143,4 +82,5 @@
     <origin xyz="0.0 0.0 0.0" rpy="0.0 0.0 0.0" />
   </joint>
+-->
   <joint name="table_joint" type="fixed">
     <parent link="table" />
@@ -148,20 +88,3 @@
     <origin xyz="0.0 0.425 0.7" rpy="0.0 0.0 1.5707" />
   </joint>
-  <!--
-  <joint name="table_column1" type="fixed">
-    <parent link="table" />
-    <child link = "column1" />
-    <origin xyz="0.45 -0.505 0.7" rpy="0.0 0.0 0.0" />
-  </joint>
-  <joint name="table_column2" type="fixed">
-    <parent link="table" />
-    <child link = "column2" />
-    <origin xyz="-0.45 -0.505 0.7" rpy="0.0 0.0 0.0" />
-  </joint>
-  <joint name="table_wp" type="fixed">
-    <parent link="table" />
-    <child link = "work_piece" />
-    <origin xyz="0.45 0.105 0.72" rpy="0.0 0.0 0.0" />
-  </joint>
-  -->
 </robot>

File: panda_table_description/urdf/table.gazebo.xacro (robot description, xacro)
@@ -1,139 +1,12 @@
 <?xml version="1.0"?>
 <robot xmlns:xacro="http://www.ros.org/wiki/xacro">
-    <xacro:macro name="panda_table_gazebo" params="robot_name:='panda' load_gripper:='true'">
-        <!-- Link0 -->
-        <gazebo reference="${robot_name}_link0">
-            <material>Gazebo/Grey</material>
-            <mu1>0.2</mu1>
-            <mu2>0.2</mu2>
-        </gazebo>
-        <!-- Link1 -->
-        <gazebo reference="${robot_name}_link1">
-            <material>Gazebo/White</material>
-            <mu1>0.2</mu1>
-            <mu2>0.2</mu2>
-        </gazebo>
-        <!-- Link2 -->
-        <gazebo reference="${robot_name}_link2">
-            <material>Gazebo/White</material>
-            <mu1>0.2</mu1>
-            <mu2>0.2</mu2>
-        </gazebo>
-        <!-- Link3 -->
-        <gazebo reference="${robot_name}_link3">
-            <material>Gazebo/White</material>
-            <mu1>0.2</mu1>
-            <mu2>0.2</mu2>
-        </gazebo>
-        <!-- Link4 -->
-        <gazebo reference="${robot_name}_link4">
-            <material>Gazebo/White</material>
-            <mu1>0.2</mu1>
-            <mu2>0.2</mu2>
-        </gazebo>
-        <!-- Link5 -->
-        <gazebo reference="${robot_name}_link5">
-            <material>Gazebo/White</material>
-            <mu1>0.2</mu1>
-            <mu2>0.2</mu2>
-        </gazebo>
-        <!-- Link6 -->
-        <gazebo reference="${robot_name}_link6">
-            <material>Gazebo/White</material>
-            <mu1>0.2</mu1>
-            <mu2>0.2</mu2>
-        </gazebo>
-        <!-- Link7 -->
-        <gazebo reference="${robot_name}_link7">
-            <material>Gazebo/Grey</material>
-            <mu1>0.2</mu1>
-            <mu2>0.2</mu2>
-            <self_collide>true</self_collide>
-        </gazebo>
-        <!-- Link8 -->
-        <gazebo reference="${robot_name}_link8">
-            <material>Gazebo/Grey</material>
-            <mu1>0.2</mu1>
-            <mu2>0.2</mu2>
-            <self_collide>true</self_collide>
-        </gazebo>
-	<xacro:if value="$(arg load_gripper)">
-        <!-- LinkHand -->
-        <gazebo reference="${robot_name}_hand">
-            <material>Gazebo/Grey</material>
-            <mu1>0.2</mu1>
-            <mu2>0.2</mu2>
-            <self_collide>true</self_collide>
-        </gazebo>
-        <!-- LinkRightFinger -->
-        <gazebo reference="${robot_name}_rightfinger">
-            <material>Gazebo/Grey</material>
-            <mu1>0.2</mu1>
-            <mu2>0.2</mu2>
-        </gazebo>
-        <!-- LinkLeftFinger -->
-        <gazebo reference="${robot_name}_leftfinger">
-            <material>Gazebo/Grey</material>
-            <mu1>0.2</mu1>
-            <mu2>0.2</mu2>
-        </gazebo>
-	</xacro:if>
-	<xacro:unless value="$(arg load_gripper)">
-        <!-- Tool -->
-        <gazebo reference="tool">
-            <material>Gazebo/Grey</material>
-            <mu1>0.2</mu1>
-            <mu2>0.2</mu2>
-            <self_collide>true</self_collide>
-            <sensor name="tool_contact_sensor" type="contact">
-      		<always_on>true</always_on>
-		<update_rate>100</update_rate>
-      		<contact>
-	            <collision>tool_collision</collision>
-                </contact>
-                <plugin name="tool_bumper" filename="libgazebo_ros_bumper.so">
-                <bumperTopicName>/panda/tool_contact_sensor_state</bumperTopicName>
-                <frameName>tool</frameName>
-                </plugin>
-            </sensor>
-        </gazebo>
-	</xacro:unless>
-	<!-- Table and columns -->
+    <xacro:macro name="table_gazebo">
+	<!-- Table -->
  	<gazebo reference="table">
-            <material>Gazebo/Grey</material>
+        <material>Gazebo/Blue</material>
             <mu1>0.2</mu1>
             <mu2>0.2</mu2>
 	    <self_collide>true</self_collide>
-        </gazebo>
- 	<gazebo reference="column1">
-            <material>Gazebo/Grey</material>
-            <mu1>0.2</mu1>
-            <mu2>0.2</mu2>
-	    <self_collide>true</self_collide>
-        </gazebo>
- 	<gazebo reference="column2">
-            <material>Gazebo/Grey</material>
-            <mu1>0.2</mu1>
-            <mu2>0.2</mu2>
-            <self_collide>true</self_collide>
-        </gazebo>
- 	<gazebo reference="mount_flange_link">
-            <material>Gazebo/Grey</material>
-            <mu1>0.2</mu1>
-            <mu2>0.2</mu2>
-        </gazebo>
- 	<gazebo reference="work_piece">
-            <material>Gazebo/Grey</material>
-            <mu1>0.2</mu1>
-            <mu2>0.2</mu2>
-	    <self_collide>true</self_collide>
-        </gazebo>
-	<!-- Box -->
- 	<gazebo reference="box">
-            <material>Gazebo/Red</material>
-            <mu1>0.2</mu1>
-            <mu2>0.2</mu2>
-	    <self_collide>true</self_collide>
-        </gazebo>
+    </gazebo>
     </xacro:macro>
 </robot>

File: panda_table_description/urdf/table.urdf.xacro (robot description, xacro)
@@ -1,52 +1,17 @@
 <?xml version="1.0"?>
-<robot xmlns:xacro="http://ros.org/wiki/xacro" name="panda" >
-  <!-- panda arm -->
-  <xacro:include filename="$(find franka_description)/robots/panda_arm.xacro"/>
-  <xacro:include filename="$(find franka_description)/robots/hand.xacro"/>
+<robot xmlns:xacro="http://ros.org/wiki/xacro" name="table" >
   <!-- for simulation -->
-  <xacro:include filename="$(find franka_description)/robots/panda.transmission.xacro"/>
-  <xacro:include filename="$(find panda_table_description)/urdf/panda_table.gazebo.xacro"/>
-  <!-- end for simulation -->
-  <xacro:panda_arm connected_to="mount_flange_link" xyz="0.0 0.0 0.0" rpy="0 0 ${pi}" />
-  <xacro:if value="$(arg load_gripper)">
-     <xacro:hand ns="panda" rpy="0 0 ${-pi/4}" connected_to="panda_link8"/>
-  </xacro:if>
-  <xacro:unless value="$(arg load_gripper)">
-   <link name="tool">
-     <inertial>
-       <mass value="0.642"/>
-       <inertia ixx="0.001" ixy="0" ixz="0" iyy="0.001" iyz="0" izz="0.001" />
-       <origin/>
-     </inertial>
-     <visual>
-       <origin xyz="0 0 -0.15" rpy="0 0 0" />
-       <geometry>
-         <cylinder radius="0.0085" length="0.3" />
-       </geometry>
-       <material name="orange"/>
-     </visual>
-     <collision name="tool_collision">
-       <origin xyz="0 0 -0.15" rpy="0 0 0" />
-       <geometry>
-         <cylinder radius="0.0085" length="0.3" />
-       </geometry>
-     </collision>
-   </link>
-     <joint name="tool_joint" type="fixed">
-       <parent link="panda_link8" />
-       <child link = "tool" />
-       <origin xyz="0.0 0.0 0.3" rpy="0.0 0.0 0.0" />
-     </joint>
-  </xacro:unless>
-  <!-- for simulation -->
-  <xacro:arg name="robot_name" default="panda"/>
-  <xacro:panda_table_gazebo robot_name="$(arg robot_name)" load_gripper="$(arg load_gripper)" />
-  <xacro:panda_transmission robot_name="$(arg robot_name)" load_gripper="$(arg load_gripper)" />
+  <xacro:include filename="$(find panda_table_description)/urdf/table.gazebo.xacro"/>
   <!-- end for simulation -->
   <link name="world" />
   <link name="table">
+    <inertial>
+      <mass value="200.0"/>
+      <inertia ixx="10.0" ixy="0" ixz="0" iyy="10.0" iyz="0" izz="10.0" />
+      <origin/>
+    </inertial>
     <visual>
       <geometry>
-	<box size="1.0 1.11 0.7" />
+	    <box size="1.0 1.11 0.7" />
       </geometry>
       <origin rpy="0 0 0" xyz="0 0 0.35" />
@@ -54,88 +19,9 @@
     <collision>
       <geometry>
-	<box size="1.0 1.11 0.7" />
+	    <box size="1.0 1.11 0.7" />
       </geometry>
       <origin rpy="0 0 0" xyz="0 0 0.35" />
     </collision>
    </link>
-   <link name="mount_flange_link">
-     <inertial>
-       <mass value="0.01"/>
-       <inertia ixx="0.001" ixy="0" ixz="0" iyy="0.001" iyz="0" izz="0.001" />
-       <origin/>
-     </inertial>
-     <visual>
-       <origin xyz="0 0 0" rpy="0 0 0" />
-       <geometry>
-         <box size="0.15 0.15 0.005" />
-       </geometry>
-       <material name="orange"/>
-     </visual>
-   </link>
-    <!--
-    <link name="box">
-     <visual>
-       <geometry>
-     <box size="0.04 0.04 0.04" />
-       </geometry>
-       <origin rpy="0 0 0" xyz="0.0 0.0 0.2575" />
-     </visual>
-     <collision>
-       <geometry>
-     <box size="0.1 0.1 0.1" />
-       </geometry>
-       <origin rpy="0 0 0" xyz="0.0 0.0 0.2575" />
-     </collision>
-    </link>
-    <joint name="table_box" type="fixed">
-      <parent link="table" />
-      <child link = "box" />
-      <origin xyz="-0.2 0.0 0.5325" rpy="0.0 0.0 0.0" />
-    </joint>
-    -->
-   <!--
-    <link name="column1">
-     <visual>
-       <geometry>
-     <box size="0.1 0.1 0.515" />
-       </geometry>
-       <origin rpy="0 0 0" xyz="0.0 0.0 0.2575" />
-     </visual>
-     <collision>
-       <geometry>
-     <box size="0.1 0.1 0.515" />
-       </geometry>
-       <origin rpy="0 0 0" xyz="0.0 0.0 0.2575" />
-     </collision>
-    </link>
-    <link name="column2">
-     <visual>
-       <geometry>
-     <box size="0.1 0.1 0.515" />
-       </geometry>
-       <origin rpy="0 0 0" xyz="0.0 0.0 0.2575" />
-     </visual>
-     <collision>
-       <geometry>
-     <box size="0.1 0.1 0.515" />
-       </geometry>
-       <origin rpy="0 0 0" xyz="0.0 0.0 0.2575" />
-     </collision>
-    </link>
-    <link name="work_piece">
-     <visual>
-       <geometry>
-     <mesh filename="package://panda_table_description/meshes/work_piece.stl" scale="0.001 0.001 0.001"/>
-       </geometry>
-       <origin rpy="0 1.5707 0" xyz="0.0 0.0 0.0" />
-     </visual>
-     <collision>
-       <geometry>
-     <mesh filename="package://panda_table_description/meshes/work_piece.stl" scale="0.001 0.001 0.001"/>
-       </geometry>
-       <origin rpy="0 1.5707 0" xyz="0.0 0.0 0.0" />
-     </collision>
-    </link>
-    -->
   <joint name="world_joint" type="fixed">
     <parent link="world" />
@@ -143,25 +29,3 @@
     <origin xyz="0.0 0.0 0.0" rpy="0.0 0.0 0.0" />
   </joint>
-  <joint name="table_joint" type="fixed">
-    <parent link="table" />
-    <child link = "mount_flange_link" />
-    <origin xyz="0.0 0.425 0.7" rpy="0.0 0.0 1.5707" />
-  </joint>
-  <!--
-  <joint name="table_column1" type="fixed">
-    <parent link="table" />
-    <child link = "column1" />
-    <origin xyz="0.45 -0.505 0.7" rpy="0.0 0.0 0.0" />
-  </joint>
-  <joint name="table_column2" type="fixed">
-    <parent link="table" />
-    <child link = "column2" />
-    <origin xyz="-0.45 -0.505 0.7" rpy="0.0 0.0 0.0" />
-  </joint>
-  <joint name="table_wp" type="fixed">
-    <parent link="table" />
-    <child link = "work_piece" />
-    <origin xyz="0.45 0.105 0.72" rpy="0.0 0.0 0.0" />
-  </joint>
-  -->
 </robot>

Commit message: fixes to the gazebo impedance controller. does not track very well, but it is certainly better. issues when starting up, beware

File: panda_table_description/urdf/panda_table.gazebo.xacro (robot description, xacro)
@@ -88,5 +88,5 @@
 	<xacro:unless value="$(arg load_gripper)">
         <!-- Tool -->
-        <gazebo reference="tool">
+	<!-- <gazebo reference="tool">
             <material>Gazebo/Grey</material>
             <mu1>0.2</mu1>
@@ -104,5 +104,11 @@
                 </plugin>
             </sensor>
-        </gazebo>
+	</gazebo> -->
+	<gazebo reference="tool">
+            <material>Gazebo/Grey</material>
+            <mu1>0.2</mu1>
+            <mu2>0.2</mu2>
+            <self_collide>true</self_collide>
+	</gazebo>
 	</xacro:unless>
 	<!-- Table and columns -->
