Commit message: Add extra urdf files

File: panda_table_description/urdf/panda_table_ramp_box.urdf.xacro (robot description, xacro)
@@ -6,5 +6,5 @@
   <!-- for simulation -->
   <xacro:include filename="$(find panda_table_description)/urdf/panda_vel.transmission.xacro"/>
-  <xacro:include filename="$(find panda_table_description)/urdf/panda_table.gazebo.xacro"/>
+  <xacro:include filename="$(find panda_table_description)/urdf/panda_table_ramp.gazebo.xacro"/>
   <!--xacro:include filename="$(find panda_table_description)/urdf/table.urdf.xacro"/-->
   <!-- end for simulation -->
@@ -73,5 +73,5 @@
     <visual>
       <geometry>
-        <box size="0.25 1 0.175" />
+        <box size="0.25 0.2775 0.175" />
       </geometry>
       <origin rpy="0 0 0" xyz="0 0 0" />
@@ -79,5 +79,5 @@
     <collision>
       <geometry>
-        <box size="0.25 1 0.175" />
+        <box size="0.25 0.2775 0.175" />
       </geometry>
       <origin rpy="0 0 0" xyz="0 0 0" />
@@ -92,5 +92,5 @@
     <visual>
       <geometry>
-        <box size="1 0.2775 0.2" />
+        <box size="0.2775 0.2775 0.2" />
       </geometry>
       <origin rpy="0 0 0" xyz="0 0 0" />
@@ -98,7 +98,34 @@
     <collision>
       <geometry>
-        <box size="1 0.2775 0.2" />
+        <box size="0.2775 0.2775 0.2" />
       </geometry>
       <origin rpy="0 0 0" xyz="0 0 0" />
+    </collision>
+  </link>
+  <link name="object_link">
+    <inertial>
+      <origin xyz="0 0 0" />
+      <mass value="10.0" />
+      <inertia ixx="0.01" ixy="0.0" ixz="0.0" iyy="0.01" iyz="0.0" izz="0.01" />
+    </inertial>
+    <visual>
+      <origin xyz="0 0 0"/>
+      <geometry>
+        <box size="0.04 0.04 0.04" />
+      </geometry>
+    </visual>
+    <collision>
+      <origin xyz="0 0 0"/>
+      <geometry>
+        <box size="0.04 0.04 0.04" />
+      </geometry>
+      <surface>
+        <friction>
+          <ode>
+            <mu>10000.0</mu>
+            <mu2>10000.0</mu2>
+          </ode>
+        </friction>
+      </surface>
     </collision>
   </link>
@@ -137,3 +164,6 @@
     <origin xyz="0.0 -0.3899 0.74395" rpy="0.0 0.0 0.0" />
   </joint>
+  <gazebo reference="object_link">
+    <material>Gazebo/Red</material>
+  </gazebo>
 </robot>

File: panda_table_description/urdf/panda_table_ramp_vel.urdf.xacro (robot description, xacro)
@@ -6,5 +6,5 @@
   <!-- for simulation -->
   <xacro:include filename="$(find panda_table_description)/urdf/panda_vel.transmission.xacro"/>
-  <xacro:include filename="$(find panda_table_description)/urdf/panda_table.gazebo.xacro"/>
+  <xacro:include filename="$(find panda_table_description)/urdf/panda_table_ramp.gazebo.xacro"/>
   <!--xacro:include filename="$(find panda_table_description)/urdf/table.urdf.xacro"/-->
   <!-- end for simulation -->
@@ -73,5 +73,5 @@
     <visual>
       <geometry>
-        <box size="0.25 1 0.175" />
+        <box size="0.25 0.2775 0.175" />
       </geometry>
       <origin rpy="0 0 0" xyz="0 0 0" />
@@ -79,5 +79,5 @@
     <collision>
       <geometry>
-        <box size="0.25 1 0.175" />
+        <box size="0.25 0.2775 0.175" />
       </geometry>
       <origin rpy="0 0 0" xyz="0 0 0" />
@@ -92,5 +92,5 @@
     <visual>
       <geometry>
-        <box size="1 0.2775 0.2" />
+        <box size="0.2775 0.2775 0.2" />
       </geometry>
       <origin rpy="0 0 0" xyz="0 0 0" />
@@ -98,5 +98,5 @@
     <collision>
       <geometry>
-        <box size="1 0.2775 0.2" />
+        <box size="0.2775 0.2775 0.2" />
       </geometry>
       <origin rpy="0 0 0" xyz="0 0 0" />
@@ -130,10 +130,10 @@
     <parent link="table" />
     <child link = "ramp" />
-    <origin xyz="0.0 -0.20 0.7" rpy="0.0 0.62 1.5708" />
+    <origin xyz="0.2 -0.20 0.7" rpy="0.0 0.62 1.5708" />
   </joint>
   <joint name="table_ramp_base_joint" type="fixed">
     <parent link="table" />
     <child link = "ramp_base" />
-    <origin xyz="0.0 -0.3899 0.74395" rpy="0.0 0.0 0.0" />
+    <origin xyz="0.2 -0.3899 0.74395" rpy="0.0 0.0 0.0" />
   </joint>
 </robot>
