Commit message: files

File: panda_table_description/urdf/box.gazebo.xacro (robot description, xacro)
@@ -5,6 +5,6 @@
  	<gazebo reference="box">
             <material>Gazebo/Red</material>
-            <mu1>0.2</mu1>
-            <mu2>0.2</mu2>
+            <mu1>10000</mu1>
+            <mu2>10000</mu2>
 	    <self_collide>true</self_collide>
     </gazebo>

File: panda_table_description/urdf/box.urdf.xacro (robot description, xacro)
@@ -13,6 +13,6 @@
         <inertial>
             <origin xyz="0 0 0" />
-            <mass value="1.0" />
-            <inertia ixx="0.001" ixy="0.0" ixz="0.0" iyy="0.001" iyz="0.0" izz="0.001" />
+            <mass value="10.0" />
+            <inertia ixx="0.01" ixy="0.0" ixz="0.0" iyy="0.01" iyz="0.0" izz="0.01" />
         </inertial>
         <visual>
@@ -27,4 +27,12 @@
                 <box size="0.04 0.04 0.04" />
             </geometry>
+            <surface>
+                <friction>
+                    <ode>
+                        <mu>10000.0</mu>
+                        <mu2>10000.0</mu2>
+                    </ode>
+                </friction>
+            </surface>
         </collision>
     </link>

File: panda_table_description/urdf/panda_table.gazebo.xacro (robot description, xacro)
@@ -107,4 +107,5 @@
 	</xacro:unless>
 	<!-- Table and columns -->
+        <!--
  	<gazebo reference="table">
             <material>Gazebo/Grey</material>
@@ -137,5 +138,7 @@
 	    <self_collide>true</self_collide>
         </gazebo>
+-->
 	<!-- Box -->
+        <!--
  	<gazebo reference="box">
             <material>Gazebo/Red</material>
@@ -144,4 +147,5 @@
 	    <self_collide>true</self_collide>
         </gazebo>
+-->
     </xacro:macro>
 </robot>

File: panda_table_description/urdf/panda_table.urdf.xacro (robot description, xacro)
@@ -7,5 +7,5 @@
   <xacro:include filename="$(find franka_description)/robots/panda.transmission.xacro"/>
   <xacro:include filename="$(find panda_table_description)/urdf/panda_table.gazebo.xacro"/>
-  <xacro:include filename="$(find panda_table_description)/urdf/table.urdf.xacro"/>
+  <!--xacro:include filename="$(find panda_table_description)/urdf/table.urdf.xacro"/-->
   <!-- end for simulation -->
   <xacro:panda_arm connected_to="mount_flange_link" xyz="0.0 0.0 0.0" rpy="0 0 ${pi}" />
@@ -45,36 +45,38 @@
   <xacro:panda_transmission robot_name="$(arg robot_name)" load_gripper="$(arg load_gripper)" />
   <!-- end for simulation -->
-  <!--
-    <link name="world" />
-    <link name="table">
-      <visual>
-        <geometry>
-      <box size="1.0 1.11 0.7" />
-        </geometry>
-        <origin rpy="0 0 0" xyz="0 0 0.35" />
-      </visual>
-      <collision>
-        <geometry>
-      <box size="1.0 1.11 0.7" />
-        </geometry>
-        <origin rpy="0 0 0" xyz="0 0 0.35" />
-      </collision>
-     </link>
-  -->
-   <link name="mount_flange_link">
-     <inertial>
-       <mass value="0.01"/>
-       <inertia ixx="0.001" ixy="0" ixz="0" iyy="0.001" iyz="0" izz="0.001" />
-       <origin/>
-     </inertial>
-     <visual>
-       <origin xyz="0 0 0" rpy="0 0 0" />
-       <geometry>
-         <box size="0.15 0.15 0.005" />
-       </geometry>
-       <material name="orange"/>
-     </visual>
-   </link>
-<!--
+  <link name="world" />
+  <link name="table">
+    <inertial>
+      <mass value="200.0"/>
+      <inertia ixx="10.0" ixy="0" ixz="0" iyy="10.0" iyz="0" izz="10.0" />
+      <origin/>
+    </inertial>
+    <visual>
+      <geometry>
+        <box size="1.0 1.11 0.7" />
+      </geometry>
+      <origin rpy="0 0 0" xyz="0 0 0.35" />
+    </visual>
+    <collision>
+      <geometry>
+        <box size="1.0 1.11 0.7" />
+      </geometry>
+      <origin rpy="0 0 0" xyz="0 0 0.35" />
+    </collision>
+  </link>
+  <link name="mount_flange_link">
+    <inertial>
+      <mass value="0.01"/>
+      <inertia ixx="0.001" ixy="0" ixz="0" iyy="0.001" iyz="0" izz="0.001" />
+      <origin/>
+    </inertial>
+    <visual>
+      <origin xyz="0 0 0" rpy="0 0 0" />
+      <geometry>
+        <box size="0.15 0.15 0.005" />
+      </geometry>
+      <material name="orange"/>
+    </visual>
+  </link>
   <joint name="world_joint" type="fixed">
     <parent link="world" />
@@ -82,5 +84,4 @@
     <origin xyz="0.0 0.0 0.0" rpy="0.0 0.0 0.0" />
   </joint>
--->
   <joint name="table_joint" type="fixed">
     <parent link="table" />

Commit message: Add urdf and launch files

File: panda_table_description/urdf/box.gazebo.xacro (robot description, xacro)
@@ -9,4 +9,10 @@
 	    <self_collide>true</self_collide>
     </gazebo>
+    <gazebo reference="object_base_link">
+        <gravity>1</gravity>
+    </gazebo>
+    <gazebo reference="object_link">
+        <material>Gazebo/Red</material>
+    </gazebo>
     </xacro:macro>
 </robot>

File: panda_table_description/urdf/box.urdf.xacro (robot description, xacro)
@@ -3,4 +3,31 @@
     <xacro:include filename="$(find panda_table_description)/urdf/box.gazebo.xacro"/>
     <link name="object_base_link">
+    </link>
+    <link name="object_link">
+        <inertial>
+            <origin xyz="0 0 0" />
+            <mass value="0.1" />
+            <inertia ixx="0.01" ixy="0.0" ixz="0.0" iyy="0.01" iyz="0.0" izz="0.01" />
+        </inertial>
+        <visual>
+            <origin xyz="0 0 0"/>
+            <geometry>
+                <box size="0.03 0.03 0.03" />
+            </geometry>
+        </visual>
+        <collision>
+            <origin xyz="0 0 0"/>
+            <geometry>
+                <box size="0.03 0.03 0.03" />
+            </geometry>
+            <surface>
+                <friction>
+                    <ode>
+                        <mu>10000</mu>
+                        <mu2>10000</mu2>
+                    </ode>
+                </friction>
+            </surface>
+        </collision>
     </link>
     <joint name="object_base_joint" type="fixed">
@@ -11,43 +38,3 @@
         <dynamics damping="0.0" friction="10.0"/>
     </joint>
-    <link name="object_link">
-        <inertial>
-            <origin xyz="0 0 0" />
-            <mass value="0.2" />
-            <inertia ixx="0.01" ixy="0.0" ixz="0.0" iyy="0.01" iyz="0.0" izz="0.01" />
-        </inertial>
-        <visual>
-            <origin xyz="0 0 0"/>
-	    <geometry>
-		    <!--
-			    <box size="0.03 0.03 0.03" />
-		<mesh filename="package://panda_table_description/meshes/rough_box.dae"/>
-		    -->
-		<mesh filename="package://panda_table_description/meshes/smooth_box.dae" scale="0.7 0.7 0.7"/>
-            </geometry>
-        </visual>
-        <collision>
-            <origin xyz="0 0 0"/>
-            <geometry>
-		    <!--
-		<box size="0.03 0.03 0.03" />
-		    -->
-		<mesh filename="package://panda_table_description/meshes/smooth_box.dae" scale="0.7 0.7 0.7"/>
-            </geometry>
-            <surface>
-                <friction>
-                    <ode>
-                        <mu>50</mu>
-                        <mu2>50</mu2>
-                    </ode>
-                </friction>
-            </surface>
-        </collision>
-    </link>
-    <gazebo reference="object_base_link">
-        <gravity>1</gravity>
-    </gazebo>
-    <gazebo reference="object_link">
-        <material>Gazebo/Red</material>
-    </gazebo>
 </robot>

File: panda_table_description/urdf/panda_table.gazebo.xacro (robot description, xacro)
@@ -144,7 +144,12 @@
 	    <self_collide>true</self_collide>
         </gazebo>
--->
+     <gazebo reference="ramp">
+            <material>Gazebo/Grey</material>
+            <mu1>0.2</mu1>
+            <mu2>0.2</mu2>
+	        <self_collide>true</self_collide>
+        <   static>true</static>
+         </gazebo>
 	<!-- Box -->
-        <!--
  	<gazebo reference="box">
             <material>Gazebo/Red</material>
@@ -153,5 +158,4 @@
 	    <self_collide>true</self_collide>
         </gazebo>
--->
     </xacro:macro>
 </robot>

Commit message: Changes to simulation environment

File: panda_table_description/urdf/box.gazebo.xacro (robot description, xacro)
@@ -3,14 +3,5 @@
     <xacro:macro name="box_gazebo">
 	<!-- Box -->
- 	<gazebo reference="box">
-            <material>Gazebo/Red</material>
-            <mu1>10000</mu1>
-            <mu2>10000</mu2>
-	    <self_collide>true</self_collide>
-    </gazebo>
-    <gazebo reference="object_base_link">
-        <gravity>1</gravity>
-    </gazebo>
-    <gazebo reference="object_link">
+    <gazebo reference="box_link">
         <material>Gazebo/Red</material>
     </gazebo>

File: panda_table_description/urdf/box.urdf.xacro (robot description, xacro)
@@ -1,8 +1,6 @@
 <?xml version="1.0"?>
-<robot xmlns:xacro="http://www.ros.org/wiki/xacro" name="simple_box">
+<robot xmlns:xacro="http://www.ros.org/wiki/xacro" name="box">
     <xacro:include filename="$(find panda_table_description)/urdf/box.gazebo.xacro"/>
-    <link name="object_base_link">
-    </link>
-    <link name="object_link">
+    <link name="box_link">
         <inertial>
             <origin xyz="0 0 0" />
@@ -38,10 +36,3 @@
         </collision>
     </link>
-    <joint name="object_base_joint" type="fixed">
-        <parent link="object_base_link"/>
-        <child link="object_link"/>
-        <axis xyz="0 0 1" />
-        <origin xyz="0 0 0" rpy="0 0 0"/>
-        <dynamics damping="0.0" friction="10.0"/>
-    </joint>
 </robot>

File: panda_table_description/urdf/panda_table.gazebo.xacro (robot description, xacro)
@@ -154,50 +154,4 @@
 	</gazebo>
 	</xacro:unless>
-	<!-- Table and columns -->
-        <!--
- 	<gazebo reference="table">
-            <material>Gazebo/Grey</material>
-            <mu1>0.2</mu1>
-            <mu2>0.2</mu2>
-	    <self_collide>true</self_collide>
-        <static>true</static>
-    </gazebo>
- 	<gazebo reference="column1">
-            <material>Gazebo/Grey</material>
-            <mu1>0.2</mu1>
-            <mu2>0.2</mu2>
-	    <self_collide>true</self_collide>
-        </gazebo>
- 	<gazebo reference="column2">
-            <material>Gazebo/Grey</material>
-            <mu1>0.2</mu1>
-            <mu2>0.2</mu2>
-            <self_collide>true</self_collide>
-        </gazebo>
- 	<gazebo reference="mount_flange_link">
-            <material>Gazebo/Grey</material>
-            <mu1>0.2</mu1>
-            <mu2>0.2</mu2>
-        </gazebo>
- 	<gazebo reference="work_piece">
-            <material>Gazebo/Grey</material>
-            <mu1>0.2</mu1>
-            <mu2>0.2</mu2>
-	    <self_collide>true</self_collide>
-        </gazebo>
-     <gazebo reference="ramp">
-            <material>Gazebo/Grey</material>
-            <mu1>0.2</mu1>
-            <mu2>0.2</mu2>
-	        <self_collide>true</self_collide>
-        <   static>true</static>
-         </gazebo>
-	<!- Box -->
- 	<gazebo reference="box">
-            <material>Gazebo/Red</material>
-            <mu1>0.2</mu1>
-            <mu2>0.2</mu2>
-	    <self_collide>true</self_collide>
-        </gazebo>
     </xacro:macro>
 </robot>
