Commit message: Add walls to simulation enviroment

File: panda_table_description/urdf/panda_table_vel.urdf.xacro (robot description, xacro)
@@ -65,4 +65,61 @@
     </collision>
   </link>
+  <link name="wall_1">
+    <inertial>
+      <mass value="200.0"/>
+      <inertia ixx="10.0" ixy="0" ixz="0" iyy="10.0" iyz="0" izz="10.0" />
+      <origin/>
+    </inertial>
+    <visual>
+      <geometry>
+        <box size="1.0 0.02 0.2" />
+      </geometry>
+      <origin rpy="0 0 0" xyz="0 0 0" />
+    </visual>
+    <collision>
+      <geometry>
+        <box size="1.0 0.02 0.2" />
+      </geometry>
+      <origin rpy="0 0 0" xyz="0 0 0" />
+    </collision>
+  </link>
+  <link name="wall_2">
+    <inertial>
+      <mass value="200.0"/>
+      <inertia ixx="10.0" ixy="0" ixz="0" iyy="10.0" iyz="0" izz="10.0" />
+      <origin/>
+    </inertial>
+    <visual>
+      <geometry>
+        <box size="0 1.11 0.2" />
+      </geometry>
+      <origin rpy="0 0 0" xyz="0 0 0" />
+    </visual>
+    <collision>
+      <geometry>
+        <box size="0 1.11 0.2" />
+      </geometry>
+      <origin rpy="0 0 0" xyz="0 0 0" />
+    </collision>
+  </link>
+  <link name="wall_3">
+    <inertial>
+      <mass value="200.0"/>
+      <inertia ixx="10.0" ixy="0" ixz="0" iyy="10.0" iyz="0" izz="10.0" />
+      <origin/>
+    </inertial>
+    <visual>
+      <geometry>
+        <box size="0 1.11 0.2" />
+      </geometry>
+      <origin rpy="0 0 0" xyz="0 0 0" />
+    </visual>
+    <collision>
+      <geometry>
+        <box size="0 1.11 0.2" />
+      </geometry>
+      <origin rpy="0 0 0" xyz="0 0 0" />
+    </collision>
+  </link>
   <link name="ramp">
     <inertial>
@@ -127,4 +184,19 @@
     <origin xyz="0.0 0.425 0.7" rpy="0.0 0.0 1.5707" />
   </joint>
+  <joint name="wall1_joint" type="fixed">
+    <parent link="table" />
+    <child link = "wall_1" />
+    <origin xyz="0.0 0.545 0.8" rpy="0.0 0.0 0.0" />
+  </joint>
+  <joint name="wall2_joint" type="fixed">
+    <parent link="table" />
+    <child link = "wall_2" />
+    <origin xyz="0.5 0.0 0.8" rpy="0.0 0.0 0.0" />
+  </joint>
+  <joint name="wall3_joint" type="fixed">
+    <parent link="table" />
+    <child link = "wall_3" />
+    <origin xyz="-0.5 0.0 0.8" rpy="0.0 0.0 0.0" />
+  </joint>
   <joint name="table_ramp_joint" type="fixed">
     <parent link="table" />
