Commit message: Add files for controller_bt task

File: panda_table_description/urdf/box.urdf.xacro (robot description, xacro)
@@ -8,10 +8,11 @@
         <child link="object_link"/>
         <axis xyz="0 0 1" />
-        <origin xyz="-0.2 0 0.72" rpy="0 0 0"/>
+        <origin xyz="0 0 0" rpy="0 0 0"/>
+        <dynamics damping="0.0" friction="10.0"/>
     </joint>
     <link name="object_link">
         <inertial>
             <origin xyz="0 0 0" />
-            <mass value="10.0" />
+            <mass value="0.1" />
             <inertia ixx="0.01" ixy="0.0" ixz="0.0" iyy="0.01" iyz="0.0" izz="0.01" />
         </inertial>
@@ -19,5 +20,5 @@
             <origin xyz="0 0 0"/>
             <geometry>
-                <box size="0.04 0.04 0.04" />
+                <box size="0.03 0.03 0.03" />
             </geometry>
         </visual>
@@ -25,11 +26,11 @@
             <origin xyz="0 0 0"/>
             <geometry>
-                <box size="0.04 0.04 0.04" />
+                <box size="0.03 0.03 0.03" />
             </geometry>
             <surface>
                 <friction>
                     <ode>
-                        <mu>10000.0</mu>
-                        <mu2>10000.0</mu2>
+                        <mu>10000</mu>
+                        <mu2>10000</mu2>
                     </ode>
                 </friction>

Commit message: playing with controller parameters

File: panda_table_description/urdf/box.urdf.xacro (robot description, xacro)
@@ -14,11 +14,15 @@
         <inertial>
             <origin xyz="0 0 0" />
-            <mass value="0.1" />
+            <mass value="0.2" />
             <inertia ixx="0.01" ixy="0.0" ixz="0.0" iyy="0.01" iyz="0.0" izz="0.01" />
         </inertial>
         <visual>
             <origin xyz="0 0 0"/>
-            <geometry>
-                <box size="0.03 0.03 0.03" />
+	    <geometry>
+		    <!--
+			    <box size="0.03 0.03 0.03" />
+		<mesh filename="package://panda_table_description/meshes/rough_box.dae"/>
+		    -->
+		<mesh filename="package://panda_table_description/meshes/smooth_box.dae" scale="0.7 0.7 0.7"/>
             </geometry>
         </visual>
@@ -26,11 +30,14 @@
             <origin xyz="0 0 0"/>
             <geometry>
-                <box size="0.03 0.03 0.03" />
+		    <!--
+		<box size="0.03 0.03 0.03" />
+		    -->
+		<mesh filename="package://panda_table_description/meshes/smooth_box.dae" scale="0.7 0.7 0.7"/>
             </geometry>
             <surface>
                 <friction>
                     <ode>
-                        <mu>10000</mu>
-                        <mu2>10000</mu2>
+                        <mu>50</mu>
+                        <mu2>50</mu2>
                     </ode>
                 </friction>

File: panda_table_description/urdf/panda_table_ramp.gazebo.xacro (robot description, xacro)
@@ -74,14 +74,56 @@
         </gazebo>
         <!-- LinkRightFinger -->
-        <gazebo reference="${robot_name}_rightfinger">
-            <material>Gazebo/Grey</material>
-            <mu1>0.2</mu1>
-            <mu2>0.2</mu2>
+	<gazebo reference="${robot_name}_rightfinger">
+	    <collision name="right_outer_collision">
+            <surface>
+            <friction>
+              <torsional>
+                <coefficient>10.0</coefficient>
+                <use_patch_radius>true</use_patch_radius>
+                <patch_radius>0.05</patch_radius>
+              </torsional>
+            </friction>
+            <contact>
+              <poissons_ratio>0.5</poissons_ratio>
+              <elastic_modulus>1e8</elastic_modulus>
+            </contact>
+            </surface>
+            </collision>
+            <mu1>10</mu1>
+            <mu2>10</mu2>
+            <maxVel>1</maxVel>
+            <kp>1000000.0</kp>
+            <kd>100.0</kd>
+            <fdir1>0 0 1</fdir1>
+            <minDepth>0.0</minDepth>
+            <maxContacts>100</maxContacts>
+            <material>Gazebo/RedBright</material>
         </gazebo>
         <!-- LinkLeftFinger -->
         <gazebo reference="${robot_name}_leftfinger">
-            <material>Gazebo/Grey</material>
-            <mu1>0.2</mu1>
-            <mu2>0.2</mu2>
+	    <collision name="left_outer_collision">
+            <surface>
+            <friction>
+              <torsional>
+                <coefficient>10.0</coefficient>
+                <use_patch_radius>true</use_patch_radius>
+                <patch_radius>0.05</patch_radius>
+              </torsional>
+            </friction>
+            <contact>
+              <poissons_ratio>0.5</poissons_ratio>
+              <elastic_modulus>1e8</elastic_modulus>
+            </contact>
+            </surface>
+            </collision>
+            <mu1>10</mu1>
+            <mu2>10</mu2>
+            <maxVel>1</maxVel>
+            <kp>1000000.0</kp>
+            <kd>100.0</kd>
+            <fdir1>0 0 1</fdir1>
+            <minDepth>0.0</minDepth>
+            <maxContacts>100</maxContacts>
+            <material>Gazebo/RedBright</material>
         </gazebo>
 	</xacro:if>

Commit message: Add finger collisions and box mesh

File: panda_table_description/urdf/box.urdf.xacro (robot description, xacro)
@@ -7,5 +7,5 @@
         <inertial>
             <origin xyz="0 0 0" />
-            <mass value="0.1" />
+            <mass value="0.2" />
             <inertia ixx="0.01" ixy="0.0" ixz="0.0" iyy="0.01" iyz="0.0" izz="0.01" />
         </inertial>
@@ -13,5 +13,9 @@
             <origin xyz="0 0 0"/>
             <geometry>
-                <box size="0.03 0.03 0.03" />
+		    <!--
+			    <box size="0.03 0.03 0.03" />
+		<mesh filename="package://panda_table_description/meshes/rough_box.dae"/>
+		    -->
+		<mesh filename="package://panda_table_description/meshes/smooth_box.dae" scale="0.5 0.5 0.5"/>
             </geometry>
         </visual>
@@ -19,11 +23,14 @@
             <origin xyz="0 0 0"/>
             <geometry>
-                <box size="0.03 0.03 0.03" />
+                <!--
+		<box size="0.03 0.03 0.03" />
+		    -->
+		<mesh filename="package://panda_table_description/meshes/smooth_box.dae" scale="0.5 0.5 0.5"/>
             </geometry>
             <surface>
                 <friction>
                     <ode>
-                        <mu>10000</mu>
-                        <mu2>10000</mu2>
+                        <mu>50</mu>
+                        <mu2>50</mu2>
                     </ode>
                 </friction>

File: panda_table_description/urdf/panda_table.gazebo.xacro (robot description, xacro)
@@ -75,13 +75,55 @@
         <!-- LinkRightFinger -->
         <gazebo reference="${robot_name}_rightfinger">
-            <material>Gazebo/Grey</material>
-            <mu1>0.2</mu1>
-            <mu2>0.2</mu2>
+	    <collision name="right_outer_collision">
+            <surface>
+            <friction>
+              <torsional>
+                <coefficient>10.0</coefficient>
+                <use_patch_radius>true</use_patch_radius>
+                <patch_radius>0.05</patch_radius>
+              </torsional>
+            </friction>
+            <contact>
+              <poissons_ratio>0.5</poissons_ratio>
+              <elastic_modulus>1e8</elastic_modulus>
+            </contact>
+            </surface>
+            </collision>
+            <mu1>10</mu1>
+            <mu2>10</mu2>
+            <maxVel>1</maxVel>
+            <kp>1000000.0</kp>
+            <kd>100.0</kd>
+            <fdir1>0 0 1</fdir1>
+            <minDepth>0.0</minDepth>
+            <maxContacts>100</maxContacts>
+            <material>Gazebo/RedBright</material>
         </gazebo>
         <!-- LinkLeftFinger -->
         <gazebo reference="${robot_name}_leftfinger">
-            <material>Gazebo/Grey</material>
-            <mu1>0.2</mu1>
-            <mu2>0.2</mu2>
+   	    <collision name="left_outer_collision">
+            <surface>
+            <friction>
+              <torsional>
+                <coefficient>10.0</coefficient>
+                <use_patch_radius>true</use_patch_radius>
+                <patch_radius>0.05</patch_radius>
+              </torsional>
+            </friction>
+            <contact>
+              <poissons_ratio>0.5</poissons_ratio>
+              <elastic_modulus>1e8</elastic_modulus>
+            </contact>
+            </surface>
+            </collision>
+            <mu1>10</mu1>
+            <mu2>10</mu2>
+            <maxVel>1</maxVel>
+            <kp>1000000.0</kp>
+            <kd>100.0</kd>
+            <fdir1>0 0 1</fdir1>
+            <minDepth>0.0</minDepth>
+            <maxContacts>100</maxContacts>
+            <material>Gazebo/RedBright</material>
         </gazebo>
 	</xacro:if>

Commit message: Change box inertias

File: panda_table_description/urdf/box.urdf.xacro (robot description, xacro)
@@ -6,5 +6,5 @@
             <origin xyz="0 0 0" />
             <mass value="0.2" />
-            <inertia ixx="0.01" ixy="0.0" ixz="0.0" iyy="0.01" iyz="0.0" izz="0.01" />
+            <inertia ixx="0.001" ixy="0.0" ixz="0.0" iyy="0.001" iyz="0.0" izz="0.001" />
         </inertial>
         <visual>
